File: boards/radio-v4.0/radio-v4.0.sch (EAGLE design)
At the start: 34 parts, among them J1 HFW8R-1ST, J2 TC2050-IDC-NL, U1 ISM43340, U2 MPM3620GQV-P, U6 TPD2E2U06DRLR, U7 TPD2E2U06DRLR, U8 TPD2E2U06DRLR

Commit message: Radio update
Connections:
- new net N$3: U$1.P49-JTAG_SEL
- new net N$4: U$1.P01-5G_RF
- net +3.3V: now also U$1.P23-VIO, U$1.P55-VBAT1, U$1.P56-VBAT2
Other:
- note added: "Datasheet says: "High to select JTAG""
- note added: "Radio Frequency in"
- note added: "STM32F405OG"
- moved on the sheet: C1, C2, C3, C4, C5, C6
