File: boards/control-v3.4/control.brd (EAGLE design)
At the start: 136.5 x 115.2 mm, 224 parts, among them IC1 MCP23017-E/SS, J1 HFW8R-1ST, J2 HFW8R-1ST, J3 6-PIN_2MM-H, J4 HFW8R-1ST, J5 2-PIN-KICKERS, J6 DF22-2, M1:C1 1uF, M1:C10 0.1uF 50V, M1:C12 ECA-1HHG221, M1:C13 ECA-1HHG221, M1:C2 1uF, M1:C3 0.022uF 50V, M1:C6 0.1uF 50V, M1:C7 0.1uF 50V, M1:C8 0.1uF 50V, M1:C9 2.2uF 50V, M1:J1 MKS-1658, M1:J2 4-PIN_2MM-H, M1:Q1 IRFH7545, M1:Q2 IRFH7545, M1:Q3 IRFH7545, M1:Q4 IRFH7545, M1:Q5 IRFH7545, M1:Q6 IRFH7545, M1:R1 10k, M1:U1 DRV8303DCA, M2:C1 1uF, M2:C10 0.1uF 50V, M2:C12 ECA-1HHG221, M2:C13 ECA-1HHG221, M2:C2 1uF, M2:C3 0.022uF 50V, M2:C6 0.1uF 50V, M2:C7 0.1uF 50V, M2:C8 0.1uF 50V, M2:C9 2.2uF 50V, M2:J1 MKS-1658, M2:J2 4-PIN_2MM-H, M2:Q1 IRFH7545, M2:Q2 IRFH7545, M2:Q3 IRFH7545, M2:Q4 IRFH7545, M2:Q5 IRFH7545, M2:Q6 IRFH7545, M2:R1 10k, M2:U1 DRV8303DCA, M3:C1 1uF, M3:C10 0.1uF 50V, M3:C12 ECA-1HHG221, M3:C13 ECA-1HHG221, M3:C2 1uF, M3:C3 0.022uF 50V, M3:C6 0.1uF 50V, M3:C7 0.1uF 50V, M3:C8 0.1uF 50V, M3:C9 2.2uF 50V, M3:J1 MKS-1658, M3:J2 4-PIN_2MM-H, M3:Q1 IRFH7545, M3:Q2 IRFH7545, M3:Q3 IRFH7545, M3:Q4 IRFH7545, M3:Q5 IRFH7545, M3:Q6 IRFH7545, M3:R1 10k, M3:U1 DRV8303DCA, M4:C1 1uF, M4:C10 0.1uF 50V, M4:C12 ECA-1HHG221, M4:C13 ECA-1HHG221, M4:C2 1uF, M4:C3 0.022uF 50V, M4:C6 0.1uF 50V, M4:C7 0.1uF 50V, M4:C8 0.1uF 50V, M4:C9 2.2uF 50V, M4:J1 MKS-1658, M4:J2 4-PIN_2MM-H, M4:Q1 IRFH7545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

Commit message: control done 3d, kicker having librarie issues
Parts:
- C23: device rcl:C0603 -> resistor:C0603

Commit message: kicker in progress
Parts:
- C23: device resistor:C0603 -> rcl:C0603
- R1, R10, R11, R12, R13, R14, R15, R2, R29, R3, R30, R32, R33, R34, R35, R4, R5, R6, R7, R8, R9: device resistor:R0603 -> rcl:R0603
