File: boards/control-v3.4/control.sch (EAGLE design)
At the start: 112 parts, among them IC1 MCP23017-E/SS, J1 HFW8R-1ST, J2 HFW8R-1ST, J3 6-PIN_2MM-H, J4 HFW8R-1ST, J5 2-PIN-KICKERS, J6 DF22-2, Q1 BSS806NH6327XTSA1, Q2 BSS806NH6327XTSA1, U1 XC3S250E-4TQG144C, U2 SN74AHC1G125, U3 MPM3620GQV-P, U4 MPM3620GQV-P, U5 VND5E006ASPTR-E, U6 MCP1824T-1202E/OT, U7 MCP1824T-2502E/OT, X1 ASV-18.432MHZ-EJ-T

Commit message: control done 3d, kicker having librarie issues
Parts:
- C23: device rcl:C-USC0603 -> resistor:C-USC0603

Commit message: kicker in progress
Parts:
- C23: device resistor:C-USC0603 -> rcl:C-USC0603
- R1, R10, R11, R12, R13, R14, R15, R2, R29, R3, R30, R32, R33, R34, R35, R4, R5, R6, R7, R8, R9: device resistor:R-US_R0603 -> rcl:R-US_R0603
