File: boards/radio-v3.2/radio-v3.2.brd (EAGLE design)
At the start: 52.5 x 50 mm, 33 parts, among them J1 HFW8R-1ST, J2 TC2050-IDC-NL, U1 ISM43340, U2 MPM3620GQV-P, U6 TPD2E2U06DRLR, U7 TPD2E2U06DRLR, U8 TPD2E2U06DRLR

Commit message: radio done, kicker in progress
Parts:
- R1, R10, R2, R5, R6, R7, R8, R9: device resistor:R0603 -> rcl:R0603
Connections:
- net !RST!_GLB: now also J2.P$10; no longer J2.10
- net +3.3V: now also J2.P$1; no longer J2.1
- net GND: now also J2.P$3, J2.P$5, J2.P$9; no longer J2.3, J2.5, J2.9
- net TCK_RAD: now also J2.P$4; no longer J2.4
- net TDI_RAD: now also J2.P$8; no longer J2.8
- net TDO_RAD: now also J2.P$6; no longer J2.6
- net TMS_RAD: now also J2.P$2; no longer J2.2
