File: boards/kicker-3.2.1/kicker.sch (EAGLE design)
At the start: 147 parts, among them J1 B2PS-VH(LF)(SN), J2 B2PS-VH(LF)(SN), J3 B2PS-VH(LF)(SN), J4 HFW8R-1ST, J5 2-PIN_2MM-H, J6 3-PIN_2MM-H, J7 !BTN_KCK_PRE_EXT, J8 !BTN_CHP_PRE_EXT, J9 !BTN_CHG_PRE_EXT, Q1 ATP302ATPAK, Q10 BSS806NSOT-23-3, Q2 IRFS4227, Q3 IXGK400N30A3, Q4 IXGK400N30A3, Q5 BSS127, Q6 AOD1N60, Q7 BSS127, Q8 BSS127, Q9 BSS127, T1 DA203X-ALDA2034, U1 MPM3620GQV-P, U2 15V, U3 LT3751FE, U4 IX4427N, U5 AT32ATQFP44, U6 ADUM7441ARQZ-RL7, U7 ADUM7441CRQZ-RL7

Commit message: control done 3d, kicker having librarie issues
Parts:
- C16: device rcl:C-USC0603 -> resistor:C-USC0603
- R2, R20, R21, R22, R23, R24, R25, R26, R27, R3, R35, R38, R39, R4, R40, R42, R43, R44, R47, R48, R49, R50, R51, R52, R53: device rcl:R-US_R0603 -> resistor:R-US_R0603
- R36, R37: device rcl:R-US_R0805 -> resistor:R-US_R0603

Commit message: kicker in progress
Parts:
- C16: device resistor:C-USC0603 -> rcl:C-USC0603
- R2, R20, R21, R22, R23, R24, R25, R26, R27, R3, R35, R37, R38, R39, R4, R40, R42, R43, R44, R47, R48, R49, R50, R51, R52, R53: device resistor:R-US_R0603 -> rcl:R-US_R0603
- R36: device resistor:R-US_R0603 -> rcl:R-US_R0805

Commit message: radio done, kicker in progress
Parts:
- C27: device rcl:C-USC0805 -> rcl:C-USC0603
- C9: device resistor:C-USC0805 -> rcl:C-USC0805
- R10, R11, R7, R8, R9: device resistor:R-US_R0805 -> rcl:R-US_R0603
- R12, R13, R14, R15: device resistor:R-US_R0805 -> rcl:R-US_R0805
- R16: device resistor:R-US_R2512 -> rcl:R-US_R2512
- R32, R36: device rcl:R-US_R0805 -> rcl:R-US_R0603
- R5, R6: device resistor:R-US_R0603 -> rcl:R-US_R0603

Commit message: kicker done, still need breakbeam and IMU
Parts:
- C19: device rcl:CPOL-USE7.5-18 -> RoboJackets-Capacitors:CPOL-USE7,5-18
- C5, C6, C7, C8: device rcl:CPOL-USE10-25 -> RoboJackets-Capacitors:CPOL-USEB25D
