File: doc/wiring-diagrams/system-diagram.sch (EAGLE design)
At the start: 1 part

Commit message: Adjused frame
Parts:
- removed KIT1: IMUIMU-KIT, RoboJackets-Boards:IMUIMU-KIT
Connections:
- removed net !CS!: KIT1.!CS!
- removed net +3.3V: KIT1.+3.3V
- removed net CLK: KIT1.SCK
- removed net GND: KIT1.GND
- removed net INT: KIT1.INT
- removed net MISO: KIT1.MISO
- removed net MOSI: KIT1.MOSI
Other:
- note removed: "Board Header Pins"
Changed lines of the file:
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@@
 <?xml version="1.0" encoding="utf-8"?>
 <!DOCTYPE eagle SYSTEM "eagle.dtd">
-<eagle version="9.5.2">
+<eagle version="9.6.2">
 <drawing>
 <settings>
-<setting alwaysvectorfont="yes"/>
+<setting alwaysvectorfont="no"/>
 <setting verticaltext="up"/>
 </settings>
@@
 <schematic xreflabel="%F%N/%S.%C%R" xrefpart="/%S.%C%R">
 <attributes>
-<attribute name="REVISION" value="1.0"/>
-<attribute name="SCH_DESC" value="Breakout board for the LSM9DS1"/>
-<attribute name="TEAM" value="RoboCup"/>
+<attribute name="REVISION" value="v1.0"/>
+<attribute name="SCH_DESC" value="High Level System Overview"/>
+<attribute name="TEAM" value="RoboCup SSL"/>
 </attributes>
 <variantdefs>
@@
 </class>
 </classes>
-<modules>
-<module name="RADIO" prefix="" dx="30.48" dy="20.32">
-<ports>
-<port name="5V" side="bottom" coord="-12.7" direction="io"/>
-<port name="GND" side="bottom" coord="-10.16" direction="io"/>
-</ports>
-<variantdefs>
-</variantdefs>
 <parts>
+<part name="FRAME1" library="RoboJackets-Frames" deviceset="FRAME_A_L" device="">
+<attribute name="REVISION" value="v1.0"/>
+<attribute name="SCH_DESC" value="High Level System Overview"/>
+<attribute name="TEAM" value="RoboCup SSL"/>
+</part>
 </parts>
 <sheets>
 <sheet>
+<description>High Level System Overview</description>
 <plain>
 </plain>
-<instances>
-</instances>
-<busses>
-</busses>
-<nets>
-</nets>
-</sheet>
-</sheets>
-</module>
-<module name="KICKER" prefix="" dx="30.48" dy="20.32">
-<ports>
-</ports>
-<variantdefs>
-</variantdefs>
-<parts>
-</parts>
-<sheets>
-<sheet>
-<plain>
-</plain>
-<instances>
-</instances>
-<busses>
-</busses>
-<nets>
-</nets>
-</sheet>
-</sheets>
-</module>
-<module name="MOTOR" prefix="" dx="30.48" dy="20.32">
-<ports>
-</ports>
-<variantdefs>
-</variantdefs>
-<parts>
-</parts>
-<sheets>
-<sheet>
-<plain>
-</plain>
-<instances>
-</instances>
-<busses>
-</busses>
-<nets>
-</nets>
-</sheet>
-</sheets>
-</module>
-<module name="CONTROL" prefix="" dx="50.8" dy="50.8">
-<ports>
-<port name="MISO_KICKER" side="left" coord="7.62" direction="io"/>
-<port name="MOSI_KICKER" side="left" coord="5.08" direction="io"/>
-<port name="SCK_KICKER" side="left" coord="2.54" direction="io"/>
-<port name="!KICKER_SELECT" side="left" coord="0" direction="io"/>
-<port name="!RESET_KICKER" side="left" coord="-2.54" direction="io"/>
-<port name="GND" side="left" coord="-5.08" direction="io"/>
-<port name="5V" side="left" coord="-7.62" direction="io"/>
-</ports>
-<variantdefs>
-</variantdefs>
-<parts>
-</parts>
-<sheets>
-<sheet>
-<plain>
-</plain>
-<instances>
-</instances>
-<busses>
-</busses>
-<nets>
-</nets>
-</sheet>
-</sheets>
-</module>
-<module name="MTRAIN" prefix="" dx="30.48" dy="20.32">
-<ports>
-</ports>
-<variantdefs>
-</variantdefs>
-<parts>
-</parts>
-<sheets>
-<sheet>
-<plain>
-</plain>
-<instances>
-</instances>
-<busses>
-</busses>
-<nets>
-</nets>
-</sheet>
-</sheets>
-</module>
-</modules>
-<parts>
-<part name="FRAME1" library="RoboJackets-Frames" deviceset="FRAME_A_L" device="">
-<attribute name="REVISION" value="1.0"/>
-<attribute name="SCH_DESC" value="High Level Connection Diagram for a Robot"/>
-<attribute name="TEAM" value="RoboCup SSL"/>
-</part>
-<part name="KIT1" library="RoboJackets-Boards" deviceset="IMU" device="IMU-KIT"/>
-<part name="GND5" library="supply1" library_urn="urn:adsk.eagle:library:371" deviceset="GND" device=""/>
-<part name="SUPPLY2" library="RoboJackets-Supplies" deviceset="+3.3V" device=""/>
-</parts>
-<sheets>
-<sheet>
-<plain>
-<wire x1="15.24" y1="175.26" x2="83.82" y2="175.26" width="0.1524" layer="97" style="shortdash"/>
-<wire x1="83.82" y1="175.26" x2="83.82" y2="137.16" width="0.1524" layer="97" style="shortdash"/>
-<wire x1="83.82" y1="137.16" x2="15.24" y2="137.16" width="0.1524" layer="97" style="shortdash"/>
-<wire x1="15.24" y1="137.16" x2="15.24" y2="175.26" width="0.1524" layer="97" style="shortdash"/>
-<text x="20.32" y="170.18" size="2.1844" layer="97">Board Header Pins</text>
-</plain>
-<moduleinsts>
-<moduleinst name="RADIO1" module="RADIO" x="104.14" y="165.1">
-<attribute name="NAME" x="104.14" y="165.1" size="2.032" layer="95" align="bottom-center"/>
-</moduleinst>
-<moduleinst name="KICKER1" module="KICKER" x="149.86" y="111.76">
-<attribute name="NAME" x="149.86" y="111.76" size="2.032" layer="95" align="bottom-center"/>
-</moduleinst>
-<moduleinst name="MOTOR1" module="MOTOR" x="73.66" y="114.3">
-<attribute name="NAME" x="73.66" y="114.3" size="2.032" layer="95" align="bottom-center"/>
-</moduleinst>
-<moduleinst name="MOTOR2" module="MOTOR" x="78.74" y="76.2">
-<attribute name="NAME" x="78.74" y="76.2" size="2.032" layer="95" align="bottom-center"/>
-</moduleinst>
-<moduleinst name="MOTOR3" module="MOTOR" x="129.54" y="78.74">
-<attribute name="NAME" x="129.54" y="78.74" size="2.032" layer="95" align="bottom-center"/>
-</moduleinst>
-<moduleinst name="MOTOR4" module="MOTOR" x="33.02" y="78.74">
-<attribute name="NAME" x="33.02" y="78.74" size="2.032" layer="95" align="bottom-center"/>
-</moduleinst>
-<moduleinst name="CONTROL1" module="CONTROL" x="193.04" y="185.42">
-<attribute name="NAME" x="193.04" y="185.42" size="2.032" layer="95" align="bottom-center"/>
-</moduleinst>
-<moduleinst name="MTRAIN1" module="MTRAIN" x="198.12" y="147.32">
-<attribute name="NAME" x="198.12" y="147.32" size="2.032" layer="95" align="bottom-center"/>
-</moduleinst>
-</moduleinsts>
 <instances>
 <instance part="FRAME1" gate="G$1" x="0" y="0" smashed="yes"/>
@@
 <attribute name="TEAM" x="173.99" y="34.29" size="3.048" layer="94" ratio="10" align="top-left"/>
 </instance>
-<instance part="KIT1" gate="G$1" x="48.26" y="154.94" smashed="yes"/>
-<instance part="GND5" gate="1" x="68.58" y="147.32" smashed="yes" rot="R90">
-<attribute name="VALUE" x="71.12" y="144.78" size="1.778" layer="96" rot="R90"/>
-</instance>
-<instance part="SUPPLY2" gate="P" x="68.58" y="162.56" smashed="yes" rot="R270">
-<attribute name="VALUE" x="71.755" y="164.465" size="1.778" layer="96" rot="R270"/>
-</instance>
 </instances>
 <busses>
 </busses>
 <nets>
-<net name="GND" class="0">
-<segment>
-<pinref part="GND5" gate="1" pin="GND"/>
-<pinref part="KIT1" gate="G$1" pin="GND"/>
-<wire x1="66.04" y1="147.32" x2="60.96" y2="147.32" width="0.1524" layer="91"/>
-</segment>
-</net>
-<net name="+3.3V" class="0">
-<segment>
-<pinref part="SUPPLY2" gate="P" pin="+3.3V"/>
-<pinref part="KIT1" gate="G$1" pin="+3.3V"/>
-<wire x1="66.04" y1="162.56" x2="60.96" y2="162.56" width="0.1524" layer="91"/>
-</segment>
-</net>
-<net name="MOSI" class="0">
-<segment>
-<pinref part="KIT1" gate="G$1" pin="MOSI"/>
-<wire x1="33.02" y1="162.56" x2="27.94" y2="162.56" width="0.1524" layer="91"/>
-<label x="27.94" y="162.56" size="1.27" layer="95" rot="R180" xref="yes"/>
-</segment>
-</net>
-<net name="MISO" class="0">
-<segment>
-<pinref part="KIT1" gate="G$1" pin="MISO"/>
-<wire x1="33.02" y1="157.48" x2="27.94" y2="157.48" width="0.1524" layer="91"/>
-<label x="27.94" y="157.48" size="1.27" layer="95" rot="R180" xref="yes"/>
-</segment>
-</net>
-<net name="CLK" class="0">
-<segment>
-<pinref part="KIT1" gate="G$1" pin="SCK"/>
-<wire x1="33.02" y1="152.4" x2="27.94" y2="152.4" width="0.1524" layer="91"/>
-<label x="27.94" y="152.4" size="1.27" layer="95" rot="R180" xref="yes"/>
-</segment>
-</net>
-<net name="INT" class="0">
-<segment>
-<label x="66.04" y="152.4" size="1.27" layer="95" xref="yes"/>
-<pinref part="KIT1" gate="G$1" pin="INT"/>
-<wire x1="60.96" y1="152.4" x2="66.04" y2="152.4" width="0.1524" layer="91"/>
-</segment>
-</net>
-<net name="!CS!" class="0">
-<segment>
-<pinref part="KIT1" gate="G$1" pin="!CS!"/>
-<wire x1="33.02" y1="147.32" x2="27.94" y2="147.32" width="0.1524" layer="91"/>
-<label x="27.94" y="147.32" size="1.27" layer="95" rot="R180" xref="yes"/>
-</segment>
-</net>
 </nets>
 </sheet>
@@
 </schematic>
 </drawing>
-<compatibility>
-<note version="8.2" severity="warning">
-Since Version 8.2, EAGLE supports online libraries. The ids
-of those online libraries will not be understood (or retained)
-with this version.
-</note>
-<note version="8.3" severity="warning">
-Since Version 8.3, EAGLE supports URNs for individual library
-assets (packages, symbols, and devices). The URNs of those assets
-will not be understood (or retained) with this version.
-</note>
-</compatibility>
 </eagle>
