File: boards/control-v3.5/control.sch (EAGLE design)
At the start: 113 parts, among them IC1 MCP23017-E/SS, J1 HFW8R-1ST, J2 HFW8R-1ST, J3 6-PIN_2MM-H, J4 HFW8R-1ST, J5 2-PIN-KICKERS, J6 DF22-2, Q1 BSS806NH6327XTSA1, Q2 BSS806NH6327XTSA1, U1 XC3S250E-4TQG144C, U2 SN74AHC1G125, U3 MPM3620GQV-P, U4 MPM3620GQV-P, U5 VND5E006ASPTR-E, U6 MCP1824T-1202E/OT, U7 MCP1824T-2502E/OT, U8 XC7A35T-1FTG256C, X1 ASV-18.432MHZ-EJ-T

Commit message: GND wired
Connections:
- net GND: now also U8G$6.GND@0, U8G$6.GND@1, U8G$6.GND@10, U8G$6.GND@11, U8G$6.GND@12, U8G$6.GND@13, U8G$6.GND@14, U8G$6.GND@15, U8G$6.GND@16, U8G$6.GND@17, U8G$6.GND@18, U8G$6.GND@19, U8G$6.GND@2, U8G$6.GND@20, U8G$6.GND@21, U8G$6.GND@22, U8G$6.GND@23, U8G$6.GND@24, U8G$6.GND@25, U8G$6.GND@26, U8G$6.GND@27, U8G$6.GND@28, U8G$6.GND@29, U8G$6.GND@3, U8G$6.GND@4, U8G$6.GND@5, U8G$6.GND@6, U8G$6.GND@7, U8G$6.GND@8, U8G$6.GND@9
Changed lines of the file:
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@@
 <part name="GND47" library="supply1" library_urn="urn:adsk.eagle:library:371" deviceset="GND" device=""/>
 <part name="U8" library="RoboJackets-ICs" deviceset="XC7A35T-1FTG256C" device=""/>
+<part name="GND50" library="supply1" deviceset="GND" device=""/>
 </parts>
 <sheets>
@@
 </sheet>
 <sheet>
-<description>FPGA</description>
+<description>FPGA IO BANKS</description>
 <plain>
 <text x="50.8" y="208.28" size="1.778" layer="97">Resistor arrays used to limit
@@
 for FPGA to check if
 battery power</text>
-<text x="320.04" y="190.5" size="1.778" layer="97">MOSI must be on p63
+<text x="312.42" y="185.42" size="1.778" layer="97">MOSI must be on p63
 and MISO must be on
 p44 for initialization by
@@
 <attribute name="VALUE" x="474.9439" y="63.366" size="1.778" layer="96"/>
 </instance>
-<instance part="U8" gate="G$4" x="723.9" y="101.6" smashed="yes">
-<attribute name="NAME" x="711.2" y="134.62" size="1.778" layer="95"/>
-<attribute name="VALUE" x="711.2" y="66.04" size="1.778" layer="95"/>
-</instance>
-<instance part="U8" gate="G$5" x="640.08" y="127" smashed="yes">
-<attribute name="NAME" x="617.22" y="142.24" size="1.778" layer="95"/>
-<attribute name="VALUE" x="617.22" y="93.98" size="1.778" layer="96"/>
-</instance>
-<instance part="U8" gate="G$6" x="728.98" y="205.74" smashed="yes">
-<attribute name="NAME" x="706.12" y="254" size="1.778" layer="95"/>
-<attribute name="VALUE" x="706.12" y="149.86" size="1.778" layer="96"/>
+<instance part="U8" gate="G$4" x="609.6" y="109.22" smashed="yes">
+<attribute name="NAME" x="596.9" y="142.24" size="1.778" layer="95"/>
+<attribute name="VALUE" x="596.9" y="73.66" size="1.778" layer="95"/>
+</instance>
+<instance part="U8" gate="G$5" x="383.54" y="220.98" smashed="yes">
+<attribute name="NAME" x="360.68" y="236.22" size="1.778" layer="95"/>
+<attribute name="VALUE" x="360.68" y="187.96" size="1.778" layer="96"/>
 </instance>
 </instances>
@@
 </segment>
 </net>
+</nets>
+</sheet>
+<sheet>
+<description>FPGA POWER AND CONTROL</description>
+<plain>
+</plain>
+<instances>
+<instance part="U8" gate="G$6" x="22.86" y="91.44" smashed="yes">
+<attribute name="NAME" x="0" y="139.7" size="1.778" layer="95"/>
+<attribute name="VALUE" x="0" y="35.56" size="1.778" layer="96"/>
+</instance>
+<instance part="GND50" gate="1" x="-12.7" y="35.56" smashed="yes">
+<attribute name="VALUE" x="-15.24" y="33.02" size="1.778" layer="96"/>
+</instance>
+</instances>
+<busses>
+</busses>
+<nets>
+<net name="GND" class="0">
+<segment>
+<pinref part="U8" gate="G$6" pin="GND@0"/>
+<pinref part="GND50" gate="1" pin="GND"/>
+<wire x1="-5.08" y1="114.3" x2="-12.7" y2="114.3" width="0.1524" layer="91"/>
+<wire x1="-12.7" y1="114.3" x2="-12.7" y2="111.76" width="0.1524" layer="91"/>
+<pinref part="U8" gate="G$6" pin="GND@1"/>
+<wire x1="-12.7" y1="111.76" x2="-12.7" y2="109.22" width="0.1524" layer="91"/>
+<wire x1="-12.7" y1="109.22" x2="-12.7" y2="106.68" width="0.1524" layer="91"/>
+<wire x1="-12.7" y1="106.68" x2="-12.7" y2="104.14" width="0.1524" layer="91"/>
+<wire x1="-12.7" y1="104.14" x2="-12.7" y2="101.6" width="0.1524" layer="91"/>
+<wire x1="-12.7" y1="101.6" x2="-12.7" y2="99.06" width="0.1524" layer="91"/>
+<wire x1="-12.7" y1="99.06" x2="-12.7" y2="96.52" width="0.1524" layer="91"/>
+<wire x1="-12.7" y1="96.52" x2="-12.7" y2="93.98" width="0.1524" layer="91"/>
+<wire x1="-12.7" y1="93.98" x2="-12.7" y2="91.44" width="0.1524" layer="91"/>
+<wire x1="-12.7" y1="91.44" x2="-12.7" y2="88.9" width="0.1524" layer="91"/>
+<wire x1="-12.7" y1="88.9" x2="-12.7" y2="86.36" width="0.1524" layer="91"/>
+<wire x1="-12.7" y1="86.36" x2="-12.7" y2="83.82" width="0.1524" layer="91"/>
+<wire x1="-12.7" y1="83.82" x2="-12.7" y2="81.28" width="0.1524" layer="91"/>
+<wire x1="-12.7" y1="81.28" x2="-12.7" y2="78.74" width="0.1524" layer="91"/>
+<wire x1="-12.7" y1="78.74" x2="-12.7" y2="76.2" width="0.1524" layer="91"/>
+<wire x1="-12.7" y1="76.2" x2="-12.7" y2="73.66" width="0.1524" layer="91"/>
+<wire x1="-12.7" y1="73.66" x2="-12.7" y2="71.12" width="0.1524" layer="91"/>
+<wire x1="-12.7" y1="71.12" x2="-12.7" y2="68.58" width="0.1524" layer="91"/>
+<wire x1="-12.7" y1="68.58" x2="-12.7" y2="66.04" width="0.1524" layer="91"/>
+<wire x1="-12.7" y1="66.04" x2="-12.7" y2="63.5" width="0.1524" layer="91"/>
+<wire x1="-12.7" y1="63.5" x2="-12.7" y2="60.96" width="0.1524" layer="91"/>
+<wire x1="-12.7" y1="60.96" x2="-12.7" y2="58.42" width="0.1524" layer="91"/>
+<wire x1="-12.7" y1="58.42" x2="-12.7" y2="55.88" width="0.1524" layer="91"/>
+<wire x1="-12.7" y1="55.88" x2="-12.7" y2="53.34" width="0.1524" layer="91"/>
+<wire x1="-12.7" y1="53.34" x2="-12.7" y2="50.8" width="0.1524" layer="91"/>
+<wire x1="-12.7" y1="50.8" x2="-12.7" y2="48.26" width="0.1524" layer="91"/>
+<wire x1="-12.7" y1="48.26" x2="-12.7" y2="45.72" width="0.1524" layer="91"/>
+<wire x1="-12.7" y1="45.72" x2="-12.7" y2="43.18" width="0.1524" layer="91"/>
+<wire x1="-12.7" y1="43.18" x2="-12.7" y2="40.64" width="0.1524" layer="91"/>
+<wire x1="-12.7" y1="40.64" x2="-12.7" y2="38.1" width="0.1524" layer="91"/>
+<wire x1="-5.08" y1="111.76" x2="-12.7" y2="111.76" width="0.1524" layer="91"/>
+<junction x="-12.7" y="111.76"/>
+<pinref part="U8" gate="G$6" pin="GND@2"/>
+<wire x1="-5.08" y1="109.22" x2="-12.7" y2="109.22" width="0.1524" layer="91"/>
+<junction x="-12.7" y="109.22"/>
+<pinref part="U8" gate="G$6" pin="GND@3"/>
+<wire x1="-5.08" y1="106.68" x2="-12.7" y2="106.68" width="0.1524" layer="91"/>
+<junction x="-12.7" y="106.68"/>
+<pinref part="U8" gate="G$6" pin="GND@4"/>
+<wire x1="-5.08" y1="104.14" x2="-12.7" y2="104.14" width="0.1524" layer="91"/>
+<junction x="-12.7" y="104.14"/>
+<pinref part="U8" gate="G$6" pin="GND@5"/>
+<wire x1="-5.08" y1="101.6" x2="-12.7" y2="101.6" width="0.1524" layer="91"/>
+<junction x="-12.7" y="101.6"/>
+<pinref part="U8" gate="G$6" pin="GND@6"/>
+<wire x1="-5.08" y1="99.06" x2="-12.7" y2="99.06" width="0.1524" layer="91"/>
+<junction x="-12.7" y="99.06"/>
+<pinref part="U8" gate="G$6" pin="GND@7"/>
+<wire x1="-5.08" y1="96.52" x2="-12.7" y2="96.52" width="0.1524" layer="91"/>
+<junction x="-12.7" y="96.52"/>
+<pinref part="U8" gate="G$6" pin="GND@8"/>
+<wire x1="-5.08" y1="93.98" x2="-12.7" y2="93.98" width="0.1524" layer="91"/>
+<junction x="-12.7" y="93.98"/>
+<pinref part="U8" gate="G$6" pin="GND@9"/>
+<wire x1="-5.08" y1="91.44" x2="-12.7" y2="91.44" width="0.1524" layer="91"/>
+<junction x="-12.7" y="91.44"/>
+<pinref part="U8" gate="G$6" pin="GND@10"/>
+<wire x1="-5.08" y1="88.9" x2="-12.7" y2="88.9" width="0.1524" layer="91"/>
+<junction x="-12.7" y="88.9"/>
+<pinref part="U8" gate="G$6" pin="GND@11"/>
+<wire x1="-5.08" y1="86.36" x2="-12.7" y2="86.36" width="0.1524" layer="91"/>
+<junction x="-12.7" y="86.36"/>
+<pinref part="U8" gate="G$6" pin="GND@12"/>
+<wire x1="-5.08" y1="83.82" x2="-12.7" y2="83.82" width="0.1524" layer="91"/>
+<junction x="-12.7" y="83.82"/>
+<pinref part="U8" gate="G$6" pin="GND@13"/>
+<wire x1="-5.08" y1="81.28" x2="-12.7" y2="81.28" width="0.1524" layer="91"/>
+<junction x="-12.7" y="81.28"/>
+<pinref part="U8" gate="G$6" pin="GND@14"/>
+<wire x1="-5.08" y1="78.74" x2="-12.7" y2="78.74" width="0.1524" layer="91"/>
+<junction x="-12.7" y="78.74"/>
+<pinref part="U8" gate="G$6" pin="GND@15"/>
+<wire x1="-5.08" y1="76.2" x2="-12.7" y2="76.2" width="0.1524" layer="91"/>
+<junction x="-12.7" y="76.2"/>
+<pinref part="U8" gate="G$6" pin="GND@16"/>
+<wire x1="-5.08" y1="73.66" x2="-12.7" y2="73.66" width="0.1524" layer="91"/>
+<junction x="-12.7" y="73.66"/>
+<pinref part="U8" gate="G$6" pin="GND@17"/>
+<wire x1="-5.08" y1="71.12" x2="-12.7" y2="71.12" width="0.1524" layer="91"/>
+<junction x="-12.7" y="71.12"/>
+<pinref part="U8" gate="G$6" pin="GND@18"/>
+<wire x1="-5.08" y1="68.58" x2="-12.7" y2="68.58" width="0.1524" layer="91"/>
+<junction x="-12.7" y="68.58"/>
+<pinref part="U8" gate="G$6" pin="GND@19"/>
+<wire x1="-5.08" y1="66.04" x2="-12.7" y2="66.04" width="0.1524" layer="91"/>
+<junction x="-12.7" y="66.04"/>
+<pinref part="U8" gate="G$6" pin="GND@20"/>
+<wire x1="-5.08" y1="63.5" x2="-12.7" y2="63.5" width="0.1524" layer="91"/>
+<junction x="-12.7" y="63.5"/>
+<pinref part="U8" gate="G$6" pin="GND@21"/>
+<wire x1="-5.08" y1="60.96" x2="-12.7" y2="60.96" width="0.1524" layer="91"/>
+<junction x="-12.7" y="60.96"/>
+<pinref part="U8" gate="G$6" pin="GND@23"/>
+<wire x1="-5.08" y1="55.88" x2="-12.7" y2="55.88" width="0.1524" layer="91"/>
+<junction x="-12.7" y="55.88"/>
+<pinref part="U8" gate="G$6" pin="GND@22"/>
+<wire x1="-5.08" y1="58.42" x2="-12.7" y2="58.42" width="0.1524" layer="91"/>
+<junction x="-12.7" y="58.42"/>
+<pinref part="U8" gate="G$6" pin="GND@24"/>
+<wire x1="-5.08" y1="53.34" x2="-12.7" y2="53.34" width="0.1524" layer="91"/>
+<junction x="-12.7" y="53.34"/>
+<pinref part="U8" gate="G$6" pin="GND@25"/>
+<wire x1="-5.08" y1="50.8" x2="-12.7" y2="50.8" width="0.1524" layer="91"/>
+<junction x="-12.7" y="50.8"/>
+<pinref part="U8" gate="G$6" pin="GND@26"/>
+<wire x1="-5.08" y1="48.26" x2="-12.7" y2="48.26" width="0.1524" layer="91"/>
+<junction x="-12.7" y="48.26"/>
+<pinref part="U8" gate="G$6" pin="GND@27"/>
+<wire x1="-5.08" y1="45.72" x2="-12.7" y2="45.72" width="0.1524" layer="91"/>
+<junction x="-12.7" y="45.72"/>
+<pinref part="U8" gate="G$6" pin="GND@28"/>
+<wire x1="-5.08" y1="43.18" x2="-12.7" y2="43.18" width="0.1524" layer="91"/>
+<junction x="-12.7" y="43.18"/>
+<pinref part="U8" gate="G$6" pin="GND@29"/>
+<wire x1="-5.08" y1="40.64" x2="-12.7" y2="40.64" width="0.1524" layer="91"/>
+<junction x="-12.7" y="40.64"/>
+</segment>
+</net>

Commit message: schematic progress
Parts:
- added C31: 330uF, rcl:CPOL-USD/7343-31R
- added C32, C33, C34, C35, C36, C37, C52, C53, C60, C73, C74, C75, C78, C79, C82, C83: 4.7uF, rcl:C-USC0603
- added C38, C39, C40, C41, C42, C43, C44, C45, C47, C48, C49, C50, C51, C61, C62, C63, C64, C65, C66, C67, C68, C69, C70, C71, C72, C76, C77, C80, C81: 0.47uF, rcl:C-USC0603
- added C46: 100uF, rcl:C-USC1210
- added C54, C55, C56, C57, C58, C59: 47uF, rcl:C-USC0805
Connections:
- new net +1.0V: C31.+, C32.1, C33.1, C34.1, C35.1, C36.1, C37.1, C38.1, C39.1, C40.1, C41.1, C42.1, C43.1, C44.1, C45.1, C46.1, C47.1, C48.1, U8G$6.VCCBRAM@0, U8G$6.VCCBRAM@1, U8G$6.VCCINT@0, U8G$6.VCCINT@1, U8G$6.VCCINT@2, U8G$6.VCCINT@3, U8G$6.VCCINT@4, U8G$6.VCCINT@5, U8G$6.VCCINT@6
- new net +1.8V: C49.1, C50.1, C51.1, C52.1, C53.1, C54.1, U8G$6.VCCAUX@0, U8G$6.VCCAUX@1, U8G$6.VCCAUX@2, U8G$6.VCCAUX@3
- new net N$10: C56.2, C61.2, C65.2, C80.2, C81.2, C82.2, C83.2
- new net N$6: C56.1, C61.1, C65.1, C80.1, C81.1, C82.1, C83.1, U8G$6.VCCO_14@0, U8G$6.VCCO_14@1, U8G$6.VCCO_14@2, U8G$6.VCCO_14@3, U8G$6.VCCO_14@4, U8G$6.VCCO_14@5
- net +3.3V: now also C55.1, C57.1, C58.1, C59.1, C60.1, C62.1, C63.1, C64.1, C66.1, C67.1, C68.1, C69.1, C70.1, C71.1, C72.1, C73.1, C74.1, C75.1, C76.1, C77.1, C78.1, C79.1, U8G$6.VCCO_0, U8G$6.VCCO_15@0, U8G$6.VCCO_15@1, U8G$6.VCCO_15@2, U8G$6.VCCO_15@3, U8G$6.VCCO_15@4, U8G$6.VCCO_15@5, U8G$6.VCCO_34@0, U8G$6.VCCO_34@1, U8G$6.VCCO_34@2, U8G$6.VCCO_35@0, U8G$6.VCCO_35@1, U8G$6.VCCO_35@2, U8G$6.VCCO_35@3, U8G$6.VCCO_35@4, U8G$6.VCCO_35@5
- net GND: now also C31.-, C32.2, C33.2, C34.2, C35.2, C36.2, C37.2, C38.2, C39.2, C40.2, C41.2, C42.2, C43.2, C44.2, C45.2, C46.2, C47.2, C48.2, C49.2, C50.2, C51.2, C52.2, C53.2, C54.2, C55.2, C57.2, C58.2, C59.2, C60.2, C62.2, C63.2, C64.2, C66.2, C67.2, C68.2, C69.2, C70.2, C71.2, C72.2, C73.2, C74.2, C75.2, C76.2, C77.2, C78.2, C79.2
Other:
- note added: "DO 1.0V AND 1,8V SUPPLY"
- note added: "VCCADC IS 1.8V, however power tree might have to be more complicated"
- note added: "VCCBATT is required only when using bitstream encryption. If battery is not used, connect VCCBATT to either ground or VCCAUX"
- moved on the sheet: U8G$5, U8G$6

Commit message: Power FPGA done, need to add missing power sources, prog fpga in progress
Parts:
- removed C10, C11, C12, C13, C14, C15, C16, C17, C19, C20, C21, C7, C9: 0.1uF, resistor:C-USC0603
- removed R10: 330, resistor:R-US_R0603
- removed R11, R9: 4.7k, resistor:R-US_R0603
- added L1, L2: 60Ohm@100MHz, RoboJackets-Inductors:FERRITE_BEAD_0603_742792602_HC
- C4: device resistor:C-USC0603 -> rcl:C-USC0603
- C6: value 0.1uF -> 0.47uF; device resistor:C-USC0603 -> rcl:C-USC0603
Connections:
- removed net +1.8V: C49.1, C50.1, C51.1, C52.1, C53.1, C54.1, U8G$6.VCCAUX@0, U8G$6.VCCAUX@1, U8G$6.VCCAUX@2, U8G$6.VCCAUX@3
- new net GNDADC: C4.2, C6.2, L1.P$1, U8G$5.VREFN, U8G$5.VREFP, U8G$6.GNDADC_0
- new net VCCAUX: C4.1, C49.1, C50.1, C51.1, C52.1, C53.1, C54.1, C6.1, L2.P$1, L2.P$2, U8G$6.VCCADC_0, U8G$6.VCCAUX@0, U8G$6.VCCAUX@1, U8G$6.VCCAUX@2, U8G$6.VCCAUX@3
- net +1.2V: no longer C10.1, C14.1, C19.1, C6.1, U1.115_VCCINT, U1.45_VCCINT, U1.80_VCCINT, U1.9_VCCINT
- net +18.5V: no longer C12.11, C13.11
- net +2.5V: no longer C15.1, C20.1, C4.1, C9.1, R10.2, R9.2, U1.102_VCCAUX, U1.137_VCCAUX, U1.30_VCCAUX, U1.65_VCCAUX
- net +3.3V: no longer C10.1, C11.1, C12.1, C13.1, C16.1, C17.1, C21.1, C7.1, R11.1, U1.100_VCCO_1, U1.121_VCCO_0, U1.138_VCCO_0, U1.13_VCCO_3, U1.28_VCCO_3, U1.42_VCCO_2, U1.49_VCCO_2, U1.79_VCCO_1
- net BST-B: no longer C7.1
- net FPGA-DONE: now also U8G$5.DONE_0; no longer R10.1, U1.72_DONE
- net FPGA-INIT: now also U8G$5.INIT_B_0; no longer R11.2, U1.40_IO_L01N_2/INIT_B
- net FPGA-PROG: now also U8G$5.PROGRAM_B_0; no longer R9.1, U1.1_PROGB
- net GND: now also L1.P$2, U8G$5.DXN_0, U8G$5.DXP_0, U8G$5.VN_0, U8G$5.VP_0, U8G$6.VCCBATT_0; no longer C10.2, C11.2, C12.2, C12.22, C13.2, C13.22, C14.2, C15.2, C16.2, C17.2, C19.2, C20.2, C21.2, C4.2, C6.2, C7.2, C9.2, U1.118_GND, U1.11_GND, U1.127_GND, U1.133_GND, U1.19_GND, U1.27_GND, U1.37_GND, U1.46_GND, U1.55_GND, U1.61_GND, U1.73_GND, U1.90_GND, U1.99_GND
- net GVDD: no longer C9.1
- net MOSI-FPGA: now also U8G$5.IO_L1P_T0_D00_MOSI_14; no longer U1.63_IO_L08N_2/DIN/D0
- net PHASE-A: no longer C7.2
- net PHASE-B: no longer C7.2
Other:
- note added: "DXP, DXN are temperaature sensing diode pins, tied to GND because it isn't used"
- note added: "Note pour moi meme : done a une circuitry speciale"
- note added: "VCCBATT is required only when using bitstream encryption. We are not using bitstream encryption therefore VCCBATT is connected to ground."
- note added: "Vp and Vn are for the analog input, if not used both should be connected to GND (page 16 XADC)"
- note removed: "VCCADC IS 1.8V, however power tree might have to be more complicated"
- note removed: "VCCBATT is required only when using bitstream encryption. If battery is not used, connect VCCBATT to either ground or VCCAUX"
- moved on the sheet: U8G$5

Commit message: Schematic progress, prog almost wired, started on io banks
Parts:
- removed C18: 0.1uF, resistor:C-USC0603
- added R10, R9: 4.7k, rcl:R-US_R0603
- added R11: 330, rcl:R-US_R0603
Connections:
- removed net R-P41: RN2.1, U1.5_IOL02N_3/VREF_3
- removed net R-P42: RN2.2, U1.4_IOL02P_3
- removed net R-P43: RN2.3, U1.3_IOL01N_3
- removed net R-P44: RN2.4, U1.2_IOL01P_3
- removed net R-P45: RN2.5, U1.142_IO_L10P_0
- removed net R-P46: RN2.6, U1.141_IP
- removed net R-P47: RN2.7, U1.140_IO_L09N_0
- removed net R-P48: RN2.8, U1.139_IO_L09P_0
- removed net R-P57: RN7.1, U1.35_IO_L10N_3
- removed net R-P58: RN7.2, U1.34_IO_L10P_3
- removed net R-P59: RN7.3, U1.32_IO_L09P_3
- removed net R-P60: RN7.4, U1.31_IO/VREF_3
- removed net R-P61: RN7.5, U1.26_IO_L08N_3
- removed net R-P62: RN7.6, U1.25_IO_L08P_3
- removed net R-P63: RN7.7, U1.24_IP
- removed net R-P64: RN7.8, U1.23_IO_L07N_3/LHCLK7
- new net +1.8V: L2.P$2
- new net T1: RN2.1, U8G$2.IO_L7P_T1_D09_14
- new net T10: RN7.2, U8G$3.IO_L7P_T1_AD2P_15
- new net T11: RN7.3, U8G$3.IO_L7N_T1_AD2N_15
- new net T12: RN7.8, U8G$3.IO_L8P_T1_AD10P_15
- new net T13: RN7.7, U8G$3.IO_L8N_T1_AD10N_15
- new net T14: RN7.6, U8G$3.IO_L9P_T1_DQS_AD3P_15
- new net T15: RN7.4, U8G$3.IO_L9N_T1_DQS_AD3N_15
- new net T16: RN7.5, U8G$3.IO_L10N_T1_AD11N_15
- new net T2: RN2.2, U8G$2.IO_L7N_T1_D10_14
- new net T3: RN2.4, U8G$2.IO_L8P_T1_D11_14
- new net T4: RN2.3, U8G$2.IO_L8N_T1_D12_14
- new net T5: RN2.6, U8G$2.IO_L9P_T1_DQS_14
- new net T6: RN2.5, U8G$2.IO_L9N_T1_DQS_D13_14
- new net T7: RN2.8, U8G$2.IO_L10P_T1_D14_14
- new net T8: RN2.7, U8G$2.IO_L10N_T1_D15_14
- new net T9: RN7.1, U8G$3.IO_L5N_T0_AD9N_15
- new net VCCO_0: C22.1, C23.1, C5.1, C55.1, C57.1, C58.1, C59.1, C60.1, C62.1, C63.1, C64.1, C66.1, C67.1, C68.1, C69.1, C70.1, C71.1, C72.1, C73.1, C74.1, C75.1, C76.1, C77.1, C78.1, C79.1, C8.1, D1.A, D10.A, D5.A, D6.A, D7.A, D8.A, D9.A, IC1.!RESET, IC1.A0, IC1.VDD, J1G$1.6, J4G$1.7, KIT2.+3.3V, R12.2, R30.2, R33.1, R5.2, R6.2, U1.143_IO_L10N_0/HSWAP, U2G2.P$V+, U6.!SHDN, U6.V_IN, U7.!SHDN, U7.V_IN, U8G$6.VCCO_0, U8G$6.VCCO_15@0, U8G$6.VCCO_15@1, U8G$6.VCCO_15@2, U8G$6.VCCO_15@3, U8G$6.VCCO_15@4, U8G$6.VCCO_15@5, U8G$6.VCCO_34@0, U8G$6.VCCO_34@1, U8G$6.VCCO_34@2, U8G$6.VCCO_35@0, U8G$6.VCCO_35@1, U8G$6.VCCO_35@2, U8G$6.VCCO_35@3, U8G$6.VCCO_35@4, U8G$6.VCCO_35@5, X1.EN, X1.VDD
- net !CS!-FPGA: now also U8G$2.IO_0_14; no longer U1.69_IP
- net +3.3V: now also R10.2, R11.2, R9.2, U8G$5.CFGBVS_0, U8G$5.M0_0, U8G$5.M1_0, U8G$5.M2_0; no longer C18.1, C22.1, C23.1, C5.1, C55.1, C57.1, C58.1, C59.1, C60.1, C62.1, C63.1, C64.1, C66.1, C67.1, C68.1, C69.1, C70.1, C71.1, C72.1, C73.1, C74.1, C75.1, C76.1, C77.1, C78.1, C79.1, C8.1, D1.A, D10.A, D5.A, D6.A, D7.A, D8.A, D9.A, IC1.!RESET, IC1.A0, IC1.VDD, J1G$1.6, J4G$1.7, KIT2.+3.3V, R12.2, R30.2, R33.1, R5.2, R6.2, U1.143_IO_L10N_0/HSWAP, U1.57_IP_L06N_2/M2/GCLK1, U1.60_IO/M1, U1.62_IO_L08P_2/M0, U1.64_VCCO_2, U2G2.P$V+, U6.!SHDN, U6.V_IN, U7.!SHDN, U7.V_IN, U8G$6.VCCO_0, U8G$6.VCCO_15@0, U8G$6.VCCO_15@1, U8G$6.VCCO_15@2, U8G$6.VCCO_15@3, U8G$6.VCCO_15@4, U8G$6.VCCO_15@5, U8G$6.VCCO_34@0, U8G$6.VCCO_34@1, U8G$6.VCCO_34@2, U8G$6.VCCO_35@0, U8G$6.VCCO_35@1, U8G$6.VCCO_35@2, U8G$6.VCCO_35@3, U8G$6.VCCO_35@4, U8G$6.VCCO_35@5, X1.EN, X1.VDD
- net FPGA-DONE: now also R11.1
- net FPGA-INIT: now also R9.1
- net FPGA-PROG: now also R10.1
- net GND: now also U8G$5.IO_L3P_TO_DQS_PUDC_B_14; no longer C18.2
- net MISO-FPGA: now also U8G$5.IO_L1P_T0_D00_MOSI_14; no longer U1.44_IO_L02N_2/MOSI/CSI_B
- net MOSI-FPGA: now also U8G$5.IO_L1N_T0_D01_DIN_14; no longer U8G$5.IO_L1P_T0_D00_MOSI_14
- net SCK-FPGA: now also U8G$5.CCLK_0; no longer U1.71_IO_L10N_2/CCLK
- net VCCAUX: no longer L2.P$2
Other:
- note added: "EMCCLK Left floating as mentionned in SPI Master config"
- note added: "We are using serial slave for the FPGA as there isn't SPI slave. We are then using an unpopulated ball for MISO, we choose the MOSI pin for master SPI config as it is close to the other pin. We will still use SPI after booting."
- note removed: "MOSI must be on p63 and MISO must be on p44 for initialization by serial from MTrain"
- note removed: "Note pour moi meme : done a une circuitry speciale"
- moved on the sheet: RN2, RN7, U8G$2

Commit message: IOs for motors all linked, still need external clock, power line and battery status wiring
Parts:
- removed C5, C8: 0.1uF, resistor:C-USC0603
Connections:
- removed net R-P1: RN8.1, U1.82_IO_L03N_1/A11
- removed net R-P10: RN6.2, U1.89_IP
- removed net R-P11: RN6.3, U1.88_IO_L05N_1/A7/RHCLK3
- removed net R-P12: RN6.4, U1.87_IO_L05P_1/A8/RHCLK2
- removed net R-P13: RN6.5, U1.86_IO_L04N_1/A9/RHCLK1
- removed net R-P14: RN6.6, U1.85_IO_L04P_1/A10/RHCLK0
- removed net R-P15: RN6.7, U1.84_IP
- removed net R-P16: RN6.8, U1.83_IO/VREF_1
- removed net R-P17: RN5.1, U1.101_IP
- removed net R-P18: RN5.2, U1.98_IO/A0
- removed net R-P19: RN5.3, U1.97_IO_L08N_1/A1
- removed net R-P2: RN8.2, U1.81_IO_L03P_1/A12
- removed net R-P20: RN5.4, U1.96_IO_L08P_1/A2
- removed net R-P21: RN5.5, U1.95_IP/VREF_1
- removed net R-P22: RN5.6, U1.94_IO_L07N_1/A3/RHCLK7
- removed net R-P23: RN5.7, U1.93_IO_L07P_1/A4/RHCLK6
- removed net R-P24: RN5.8, U1.92_IO_L06N_1/A5/RHCLK5
- removed net R-P25: RN3.1, U1.117_IO_L02N_0
- removed net R-P26: RN3.2, U1.116_IO_L02P_0
- removed net R-P27: RN3.3, U1.113_IO_L01N_0
- removed net R-P28: RN3.4, U1.112_IO_L01P_0
- removed net R-P29: RN3.5, U1.106_IO_L10N_1/LDC2
- removed net R-P3: RN8.3, U1.77_IO_L02N_1/A13
- removed net R-P30: RN3.6, U1.105_IO_L10P_1/LDC1
- removed net R-P31: RN3.7, U1.104_IO_L09N_1/LDC0
- removed net R-P32: RN3.8, U1.103_IO_L09P_1/HDC
- removed net R-P36: RN1.4, U1.125_IO_L05P_0/GCLK6
- removed net R-P37: RN1.5, U1.124_IO/VREF_0
- removed net R-P38: RN1.6, U1.123_IO_L04N_0/GCLK5
- removed net R-P39: RN1.7, U1.122_IO_L04P_0/GCLK4
- removed net R-P4: RN8.4, U1.76_IO_L02P_1/A14
- removed net R-P40: RN1.8, U1.119_IP_L03P_0
- removed net R-P49: RN4.1, U1.21_IO_L06N_3/LHCLK5
- removed net R-P5: RN8.5, U1.75_IO_L01N_1/A15
- removed net R-P50: RN4.2, U1.20_IO_L06P_3/LHCLK4
- removed net R-P51: RN4.3, U1.17_IO_L05N_3/LHCLK3
- removed net R-P52: RN4.4, U1.16_IO_L05P_3/LHCLK2
- removed net R-P53: RN4.5, U1.15_IO_L04N_3/LHCLK1
- removed net R-P54: RN4.6, U1.14_IO_L04P_3/LHCLK0
- removed net R-P55: RN4.7, U1.8_IOL03N_3
- removed net R-P56: RN4.8, U1.7_IOL03P_3
- removed net R-P6: RN8.6, U1.74_IO_L01P_1/A16
- removed net R-P7: RN8.7, U1.70_IO_L10P_2/VS0/A17
- removed net R-P8: RN8.8, U1.68_IO_L09N_2/VS1/A18
- removed net R-P9: RN6.1, U1.91_IO_L06P_1/A6/RHCLK4
- new net T17: RN4.8, U8G$3.IO_L23N_T3_FWE_B_15
- new net T18: RN4.7, U8G$3.IO_L23P_T3_FOE_B_15
- new net T19: RN4.5, U8G$3.IO_L22N_T3_A16_15
- new net T20: RN4.6, U8G$3.IO_L22P_T3_A17_15
- new net T21: RN4.2, U8G$3.IO_L18N_T2_A23_15
- new net T22: RN4.4, U8G$3.IO_L18P_T2_A24_15
- new net T23: RN4.1, U8G$3.IO_L17N_T2_A25_15
- new net T24: RN4.3, U8G$3.IO_L17P_T2_A26_15
- new net T25: RN8.8, U8G$1.IO_L3P_T0_DQS_AD5P_35
- new net T26: RN8.7, U8G$1.IO_L3N_T0_DQS_AD5N_35
- new net T27: RN8.6, U8G$1.IO_L4N_T0_35
- new net T28: RN8.2, U8G$1.IO_L7N_T1_AD6N_35
- new net T29: RN8.4, U8G$1.IO_L8P_T1_AD14P_35
- new net T30: RN8.5, U8G$1.IO_L8N_T1_AD14N_35
- new net T31: RN8.1, U8G$1.IO_L9P_T1_DQS_AD7P_35
- new net T32: RN8.3, U8G$1.IO_L9N_T1_DQS_AD7N_35
- new net T33: RN6.8, U8G$1.IO_L7P_T1_AD6P_35
- new net T34: RN6.6, U8G$1.IO_L10P_T1_AD15P_35
- new net T35: RN6.7, U8G$1.IO_L10N_T1_AD15N_35
- new net T36: RN6.1, U8G$1.IO_L20N_T3_35
- new net T37: RN6.2, U8G$1.IO_L17N_T2_35
- new net T38: RN6.3, U8G$1.IO_L17P_T2_35
- new net T39: RN6.5, U8G$1.IO_L15N_T2_DQS_35
- new net T40: RN6.4, U8G$1.IO_L15P_T2_DQS_35
- new net T41: RN5.6, U8G$1.IO_L24N_T3_35
- new net T42: RN5.4, U8G$1.IO_L23N_T3_35
- new net T43: RN5.7, U8G$1.IO_L22N_T3_35
- new net T44: RN5.5, U8G$1.IO_L22P_T3_35
- new net T45: RN5.8, U8G$1.IO_L20P_T3_35
- new net T46: RN5.3, U8G$4.IO_L2P_T0_34
- new net T47: RN5.2, U8G$4.IO_L2N_T0_34
- new net T48: RN5.1, U8G$4.IO_L4P_T0_34
- new net T49: RN3.2, U8G$4.IO_L9N_T1_DQS_34
- new net T50: RN3.1, U8G$4.IO_L9P_T1_DQS_34
- new net T51: RN3.3, U8G$4.IO_L8N_T1_34
- new net T52: RN3.4, U8G$4.IO_L8P_T1_34
- new net T53: RN3.5, U8G$4.IO_L7N_T1_34
- new net T54: RN3.6, U8G$4.IO_L7P_T1_34
- new net T55: RN3.7, U8G$4.IO_L4N_T0_34
- new net T56: RN3.8, U8G$4.IO_L3N_T0_DQS_34
- new net T57: RN1.8, U8G$2.IO_L23N_T3_A02_D18_14
- new net T58: RN1.4, U8G$2.IO_L22N_T3_A04_D20_14
- new net T59: RN1.5, U8G$2.IO_L22P_T3_A05_D21_14
- new net T60: RN1.6, U8G$2.IO_L21N_T3_DQS_A06_D22_14
- new net T61: RN1.7, U8G$2.IO_L21P_T3_DQS_14
- net BATT-FPGA: no longer U1.136_IP
- net BST-C: no longer C8.1
- net GND: no longer C5.2, C8.2
- net PHASE-C: no longer C8.2
- net VCCO_0: no longer C5.1, C8.1, U1.143_IO_L10N_0/HSWAP
Other:
- note added: "IO DONE, NEED 50MgH clock , do power lines for fpga, check how power voltage is monitored, clean up schematic. Other stuff not thought about ?"
- moved on the sheet: RN1, RN3, RN4, RN5, RN6, RN8, U8G$4
