File: boards/control-v3.5/control.sch (EAGLE design)
At the start: 152 parts, among them IC1 MCP23017-E/SS, J1 HFW8R-1ST, J2 HFW8R-1ST, J3 6-PIN_2MM-H, J4 HFW8R-1ST, J5 2-PIN-KICKERS, J6 DF22-2, Q1 BSS806NH6327XTSA1, Q2 BSS806NH6327XTSA1, U1 XC3S250E-4TQG144C, U2 SN74AHC1G125, U3 MPM3620GQV-P, U4 MPM3620GQV-P, U5 VND5E006ASPTR-E, U6 MCP1824T-1202E/OT, U7 MCP1824T-2502E/OT, U8 XC7A35T-1FTG256C, X1 ASV-18.432MHZ-EJ-T

Commit message: Organized IOs, new clock missing, adding power lines
Parts:
- removed C3: 0.1uF, resistor:C-USC0603
- removed R7: 68k, resistor:R-US_R0603
- removed R8: 10k, resistor:R-US_R0603
- removed U1: XC3S250E-4TQG144C, RoboJackets-ICs:XC3S250E-4TQG144C
Connections:
- removed net !CS: U1.!SCS
- removed net !FAULT: U1.!FAULT
- removed net !OCTW: U1.!OCTW
- removed net A-H: U1.INH_A, U1.INH_B
- removed net A-L: U1.INL_A, U1.INL_B
- removed net B-H: U1.INH_A, U1.INH_B
- removed net B-L: U1.INL_A, U1.INL_B
- removed net BATT-FPGA: C3.1, R7.2, R8.1
- removed net BST-B: U1.BST_B
- removed net BST-C: U1.BST_C
- removed net C-H: U1.INH_C
- removed net C-L: U1.INL_C
- removed net CP1: C3.1, U1.CP1
- removed net CP2: C3.2, U1.CP2
- removed net FPGA-CLK: U1.50_IO_L04P_2/D7/GCLK12, X1.OUT
- removed net GH-B: U1.GH_B
- removed net GH-C: U1.GH_C
- removed net GL-B: U1.GL_B
- removed net GL-C: U1.GL_C
- removed net GVDD: U1.GVDD
- removed net SO1: U1.SO1
- removed net SO2: U1.SO2
- net +18.5V: no longer R7.1, U1.PVDD
- net +3.3V: no longer U1.DVDD, U1.REF, U1.VDD_SPI
- net AVDD: no longer U1.AVDD
- net BST-A: no longer U1.BST_A
- net EN-GATE: no longer U1.EN_GATE
- net GH-A: no longer U1.GH_A
- net GL-A: no longer U1.GL_A
- net GND: no longer C3.2, R8.2, U1.AGND, U1.DC_CAL, U1.DTC, U1.GND, U1.REF, U1.SL_A, U1.SL_B, U1.SL_C
- net MISO: no longer U1.SDO
- net MOSI: no longer U1.SDI
- net PHASE-A: no longer U1.SH_A, U1.SH_B
- net PHASE-B: no longer U1.SH_A, U1.SH_B
- net PHASE-C: no longer U1.SH_C
- net SCK: no longer U1.SCLK
Other:
- note added: "DD/M1"
- note added: "IO BANK 14 FPGA"
- note added: "IO BANK 15 FPGA"
- note added: "IO BANK 34 FPGA"
- note added: "IO BANK 35 FPGA"
- note added: "M1/M2"
- note added: "M2/M3"
- note added: "M3/M4"
- note removed: "Voltage divider on 18.5v for FPGA to check if battery power"
- moved on the sheet: C22, RN1, RN2, RN3, RN4, RN5, RN6, RN7, RN8, U8G$1, U8G$2, U8G$3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
