File: boards/control-v3.5/control.sch (EAGLE design)
At the start: 148 parts, among them IC1 MCP23017-E/SS, J1 HFW8R-1ST, J2 HFW8R-1ST, J3 6-PIN_2MM-H, J4 HFW8R-1ST, J5 2-PIN-KICKERS, J6 DF22-2, Q1 BSS806NH6327XTSA1, Q2 BSS806NH6327XTSA1, U2 SN74AHC1G125, U3 MPM3620GQV-P, U4 MPM3620GQV-P, U5 VND5E006ASPTR-E, U6 MCP1824T-1202E/OT, U7 MCP1824T-2502E/OT, U8 XC7A35T-1FTG256C, X1 ASV-18.432MHZ-EJ-T

Commit message: cleanup
Other:
- note added: "Power FPGA"
- note added: "Prog FPGA"
- moved on the sheet: C31, C32, C33, C34, C35, C36, C37, C38, C39, C4, C40, C41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

Commit message: FPGA board schematic ready for review!
Parts:
- removed C29: 2.2uF 50V, resistor:C-USC0603
- removed D5: RED, RoboJackets-LEDs:LED-SMD-RED
- removed R34: 0, resistor:R-US_R0603
- removed U6: MCP1824T-1202E/OT, RoboJackets-PowerICs:MCP1824T-1202E/OT
- removed U7: MCP1824T-2502E/OT, RoboJackets-PowerICs:MCP1824T-2502E/OT
- added C3, C8: 1uF, resistor:C-USC0603
- added C5, C7: 1uF X7R, resistor:C-USC0603
- added R7: 0, resistor:R-US_R0603
- added U$17: MIC47100-1.0YML-TR, RoboJackets-PowerICs:MIC47100-1.0YML-TR
- added U1: MCP1824T-1802E/OT, RoboJackets-PowerICs:MCP1824T-1802E/OT
- X1: value ASV-18.432MHZ-EJ-T -> ASV-50.000MHZ-E-T; device RoboJackets-FreqGen:ASV-18.432MHZ-EJ-T -> RoboJackets-FreqGen:ASV-50.000MHZ-E-T
Connections:
- removed net +1.2V: R34.2
- removed net +1.2V-PRE: C29.1, R34.1, U6.V_OUT
- removed net +2.5V: R35.2
- removed net +2.5V-PRE: C30.1, R35.1, U7.V_OUT
- new net !CS: U1.!SCS
- new net !FAULT: U1.!FAULT
- new net !OCTW: U1.!OCTW
- new net A-H: U1.INH_A, U1.INH_B
- new net A-L: U1.INL_A, U1.INL_B
- new net B-H: U1.INH_A, U1.INH_B
- new net B-L: U1.INL_A, U1.INL_B
- new net BST-B: C7.1, U1.BST_B
- new net BST-C: C8.1, U1.BST_C
- new net C-H: U1.INH_C
- new net C-L: U1.INL_C
- new net CP1: C3.1, U1.CP1
- new net CP2: C3.2, U1.CP2
- new net EXT_SCK: U8G$3.IO_L2N_T0_AD8N_15, X1.OUT
- new net GH-B: U1.GH_B
- new net GH-C: U1.GH_C
- new net GL-B: U1.GL_B
- new net GL-C: U1.GL_C
- new net GVDD: U1.GVDD
- new net N$3: C5.1, R7.1, U$17.FB/ADJ, U$17.OUT@0, U$17.OUT@1
- new net SO1: U1.SO1
- new net SO2: U1.SO2
- new net V_OUT: C30.1, R35.1, U1.V_OUT
- net +1.0V: now also R7.2
- net +1.8V: now also R35.2
- net +18.5V: now also U1.PVDD
- net +3.3V: now also C3.1, C7.1, C8.1, U$17.BIAS, U$17.EN, U$17.IN@0, U1.DVDD, U1.REF, U1.VDD_SPI
- net AVDD: now also U1.AVDD
- net BST-A: now also U1.BST_A
- net EN-GATE: now also U1.EN_GATE
- net GH-A: now also U1.GH_A
- net GL-A: now also U1.GL_A
- net GND: now also C3.2, C5.2, C7.2, C8.2, U$17.GND, U1.AGND, U1.DC_CAL, U1.DTC, U1.GND, U1.REF, U1.SL_A, U1.SL_B, U1.SL_C; no longer C29.2, U6.GND, U7.GND
- net MISO: now also U1.SDO
- net MOSI: now also U1.SDI
- net PHASE-A: now also C7.2, U1.SH_A, U1.SH_B
- net PHASE-B: now also C7.2, U1.SH_A, U1.SH_B
- net PHASE-C: now also C8.2, U1.SH_C
- net PWR-ERR: now also U1.PWRGD; no longer D5.K, U6.PWRGD, U7.PWRGD
- net SCK: now also U1.SCLK
- net VCCO_0: now also U1.!SHDN, U1.V_IN; no longer D5.A, U6.!SHDN, U6.V_IN, U7.!SHDN, U7.V_IN
Other:
- note added: "1.0V Reg"
- note added: "1.8V Reg"
- note added: "External Clock"
- note added: "This part is fixed so pin 6 is FB"
- note added: "When 1.8v out of tolerance ERR LED turns on"
- note removed: "1.2V Reg"
- note removed: "2.5V Reg"
- note removed: "DO 1.0V AND 1,8V SUPPLY"
- note removed: "IO DONE, NEED 50MgH clock , do power lines for fpga, check how power voltage is monitored, clean up schematic. Other stuff not thought about ?"
- note removed: "When 1.2v or 2.5v or out of tolerance ERR LED turns on"
- moved on the sheet: C22, X1

Commit message: some modif
Connections:
- net !CS!-IR renamed !CS!-WHISKERS
- net !CS!-RAD0 renamed !CS!-RADIO
- net !RST!-IR renamed !RST!-WHISKERS
- net INT-RAD0 renamed INT-RADIO
- removed net N$10: C56.2, C61.2, C65.2, C80.2, C81.2, C82.2, C83.2
- removed net N$6: C56.1, C61.1, C65.1, C80.1, C81.1, C82.1, C83.1, U8G$6.VCCO_14@0, U8G$6.VCCO_14@1, U8G$6.VCCO_14@2, U8G$6.VCCO_14@3, U8G$6.VCCO_14@4, U8G$6.VCCO_14@5
- net +3.3V: now also C56.1, C61.1, C65.1, C80.1, C81.1, C82.1, C83.1, U8G$6.VCCO_14@0, U8G$6.VCCO_14@1, U8G$6.VCCO_14@2, U8G$6.VCCO_14@3, U8G$6.VCCO_14@4, U8G$6.VCCO_14@5
- net GND: now also C56.2, C61.2, C65.2, C80.2, C81.2, C82.2, C83.2
Changed lines of the file:
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@@
 <part name="FRAME2" library="RoboJackets-Frames" deviceset="FRAME_B_L" device="">
 <attribute name="REVISION" value="v3.4"/>
-<attribute name="SCH_DESC" value="FPGA"/>
+<attribute name="SCH_DESC" value="FPGA IO banks"/>
 </part>
 <part name="R1" library="resistor" library_urn="urn:adsk.eagle:library:348" deviceset="R-US_" device="R0603" package3d_urn="urn:adsk.eagle:package:23555/2" value="68k 1%"/>
@@
 <part name="FRAME8" library="RoboJackets-Frames" deviceset="FRAME_B_L" device="">
 <attribute name="REVISION" value="v3.4"/>
-<attribute name="SCH_DESC" value="FPGA"/>
+<attribute name="SCH_DESC" value="FPGA power and control"/>
 </part>
 <part name="X1" library="RoboJackets-FreqGen" deviceset="ASV-*" device="" technology="50.000MHZ-E-T"/>
@@
 </segment>
 </net>
-<net name="!CS!-RAD0" class="0">
+<net name="!CS!-RADIO" class="0">
 <segment>
 <pinref part="KIT1" gate="G$1" pin="P17"/>
@@
 </segment>
 </net>
-<net name="INT-RAD0" class="0">
+<net name="INT-RADIO" class="0">
 <segment>
 <pinref part="KIT1" gate="G$1" pin="P30"/>
@@
 </segment>
 </net>
-<net name="!RST!-IR" class="0">
+<net name="!RST!-WHISKERS" class="0">
 <segment>
 <pinref part="KIT1" gate="G$1" pin="P9"/>
@@
 </segment>
 </net>
-<net name="!CS!-IR" class="0">
+<net name="!CS!-WHISKERS" class="0">
 <segment>
 <pinref part="KIT1" gate="G$1" pin="P10"/>
@@
 <wire x1="-22.86" y1="7.62" x2="-20.32" y2="7.62" width="0.1524" layer="91"/>
 </segment>
-</net>
-<net name="N$6" class="0">
 <segment>
-<pinref part="U8" gate="G$6" pin="VCCO_14@5"/>
-<wire x1="17.78" y1="93.98" x2="20.32" y2="93.98" width="0.1524" layer="91"/>
-<wire x1="20.32" y1="93.98" x2="20.32" y2="96.52" width="0.1524" layer="91"/>
-<pinref part="U8" gate="G$6" pin="VCCO_14@0"/>
-<wire x1="20.32" y1="96.52" x2="20.32" y2="99.06" width="0.1524" layer="91"/>
-<wire x1="20.32" y1="99.06" x2="20.32" y2="101.6" width="0.1524" layer="91"/>
-<wire x1="20.32" y1="101.6" x2="20.32" y2="104.14" width="0.1524" layer="91"/>
-<wire x1="20.32" y1="104.14" x2="20.32" y2="106.68" width="0.1524" layer="91"/>
-<wire x1="20.32" y1="106.68" x2="17.78" y2="106.68" width="0.1524" layer="91"/>
-<pinref part="U8" gate="G$6" pin="VCCO_14@1"/>
-<wire x1="17.78" y1="104.14" x2="20.32" y2="104.14" width="0.1524" layer="91"/>
-<junction x="20.32" y="104.14"/>
-<pinref part="U8" gate="G$6" pin="VCCO_14@2"/>
-<wire x1="17.78" y1="101.6" x2="20.32" y2="101.6" width="0.1524" layer="91"/>
-<junction x="20.32" y="101.6"/>
-<pinref part="U8" gate="G$6" pin="VCCO_14@3"/>
-<wire x1="17.78" y1="99.06" x2="20.32" y2="99.06" width="0.1524" layer="91"/>
-<junction x="20.32" y="99.06"/>
-<pinref part="U8" gate="G$6" pin="VCCO_14@4"/>
-<wire x1="17.78" y1="96.52" x2="20.32" y2="96.52" width="0.1524" layer="91"/>
-<junction x="20.32" y="96.52"/>
-<pinref part="C61" gate="G$1" pin="1"/>
-<wire x1="20.32" y1="106.68" x2="25.4" y2="106.68" width="0.1524" layer="91"/>
-<junction x="20.32" y="106.68"/>
-<pinref part="C65" gate="G$1" pin="1"/>
-<wire x1="25.4" y1="106.68" x2="35.56" y2="106.68" width="0.1524" layer="91"/>
-<junction x="25.4" y="106.68"/>
-<pinref part="C80" gate="G$1" pin="1"/>
-<wire x1="35.56" y1="106.68" x2="45.72" y2="106.68" width="0.1524" layer="91"/>
-<junction x="35.56" y="106.68"/>
-<pinref part="C81" gate="G$1" pin="1"/>
-<wire x1="45.72" y1="106.68" x2="55.88" y2="106.68" width="0.1524" layer="91"/>
-<junction x="45.72" y="106.68"/>
-<pinref part="C82" gate="G$1" pin="1"/>
-<wire x1="55.88" y1="106.68" x2="66.04" y2="106.68" width="0.1524" layer="91"/>
-<junction x="55.88" y="106.68"/>
-<pinref part="C83" gate="G$1" pin="1"/>
-<wire x1="66.04" y1="106.68" x2="73.66" y2="106.68" width="0.1524" layer="91"/>
-<junction x="66.04" y="106.68"/>
-<pinref part="C56" gate="G$1" pin="1"/>
-<wire x1="73.66" y1="106.68" x2="81.28" y2="106.68" width="0.1524" layer="91"/>
-<junction x="73.66" y="106.68"/>
+<pinref part="C61" gate="G$1" pin="2"/>
+<pinref part="C65" gate="G$1" pin="2"/>
+<wire x1="25.4" y1="99.06" x2="35.56" y2="99.06" width="0.1524" layer="91"/>
+<pinref part="C80" gate="G$1" pin="2"/>
+<wire x1="35.56" y1="99.06" x2="45.72" y2="99.06" width="0.1524" layer="91"/>
+<junction x="35.56" y="99.06"/>
+<pinref part="C81" gate="G$1" pin="2"/>
+<wire x1="45.72" y1="99.06" x2="55.88" y2="99.06" width="0.1524" layer="91"/>
+<junction x="45.72" y="99.06"/>
+<pinref part="C82" gate="G$1" pin="2"/>
+<wire x1="55.88" y1="99.06" x2="66.04" y2="99.06" width="0.1524" layer="91"/>
+<junction x="55.88" y="99.06"/>
+<pinref part="C83" gate="G$1" pin="2"/>
+<wire x1="66.04" y1="99.06" x2="73.66" y2="99.06" width="0.1524" layer="91"/>
+<junction x="66.04" y="99.06"/>
+<pinref part="C56" gate="G$1" pin="2"/>
+<wire x1="73.66" y1="99.06" x2="81.28" y2="99.06" width="0.1524" layer="91"/>
+<junction x="73.66" y="99.06"/>
+<pinref part="GND75" gate="1" pin="GND"/>
+<wire x1="81.28" y1="99.06" x2="81.28" y2="96.52" width="0.1524" layer="91"/>
+<junction x="81.28" y="99.06"/>
 </segment>
 </net>
@@
 </segment>
 </net>
-<net name="N$10" class="0">
-<segment>
-<pinref part="C61" gate="G$1" pin="2"/>
-<pinref part="C65" gate="G$1" pin="2"/>
-<wire x1="25.4" y1="99.06" x2="35.56" y2="99.06" width="0.1524" layer="91"/>
-<pinref part="C80" gate="G$1" pin="2"/>
-<wire x1="35.56" y1="99.06" x2="45.72" y2="99.06" width="0.1524" layer="91"/>
-<junction x="35.56" y="99.06"/>
-<pinref part="C81" gate="G$1" pin="2"/>
-<wire x1="45.72" y1="99.06" x2="55.88" y2="99.06" width="0.1524" layer="91"/>
-<junction x="45.72" y="99.06"/>
-<pinref part="C82" gate="G$1" pin="2"/>
-<wire x1="55.88" y1="99.06" x2="66.04" y2="99.06" width="0.1524" layer="91"/>
-<junction x="55.88" y="99.06"/>
-<pinref part="C83" gate="G$1" pin="2"/>
-<wire x1="66.04" y1="99.06" x2="73.66" y2="99.06" width="0.1524" layer="91"/>
-<junction x="66.04" y="99.06"/>
-<pinref part="C56" gate="G$1" pin="2"/>
-<wire x1="73.66" y1="99.06" x2="81.28" y2="99.06" width="0.1524" layer="91"/>
-<junction x="73.66" y="99.06"/>
-</segment>
-</net>
 <net name="VCCAUX" class="0">
 <segment>
@@
 <wire x1="40.64" y1="7.62" x2="40.64" y2="10.16" width="0.1524" layer="91"/>
 </segment>
+<segment>
+<pinref part="U8" gate="G$6" pin="VCCO_14@5"/>
+<wire x1="17.78" y1="93.98" x2="20.32" y2="93.98" width="0.1524" layer="91"/>
+<wire x1="20.32" y1="93.98" x2="20.32" y2="96.52" width="0.1524" layer="91"/>
+<pinref part="U8" gate="G$6" pin="VCCO_14@0"/>
+<wire x1="20.32" y1="96.52" x2="20.32" y2="99.06" width="0.1524" layer="91"/>
+<wire x1="20.32" y1="99.06" x2="20.32" y2="101.6" width="0.1524" layer="91"/>
+<wire x1="20.32" y1="101.6" x2="20.32" y2="104.14" width="0.1524" layer="91"/>
+<wire x1="20.32" y1="104.14" x2="20.32" y2="106.68" width="0.1524" layer="91"/>
+<wire x1="20.32" y1="106.68" x2="17.78" y2="106.68" width="0.1524" layer="91"/>
+<pinref part="U8" gate="G$6" pin="VCCO_14@1"/>
+<wire x1="17.78" y1="104.14" x2="20.32" y2="104.14" width="0.1524" layer="91"/>
+<junction x="20.32" y="104.14"/>
+<pinref part="U8" gate="G$6" pin="VCCO_14@2"/>
+<wire x1="17.78" y1="101.6" x2="20.32" y2="101.6" width="0.1524" layer="91"/>
+<junction x="20.32" y="101.6"/>
+<pinref part="U8" gate="G$6" pin="VCCO_14@3"/>
+<wire x1="17.78" y1="99.06" x2="20.32" y2="99.06" width="0.1524" layer="91"/>
+<junction x="20.32" y="99.06"/>
+<pinref part="U8" gate="G$6" pin="VCCO_14@4"/>
+<wire x1="17.78" y1="96.52" x2="20.32" y2="96.52" width="0.1524" layer="91"/>
+<junction x="20.32" y="96.52"/>
+<pinref part="C61" gate="G$1" pin="1"/>
+<wire x1="20.32" y1="106.68" x2="25.4" y2="106.68" width="0.1524" layer="91"/>
+<junction x="20.32" y="106.68"/>
+<pinref part="C65" gate="G$1" pin="1"/>
+<wire x1="25.4" y1="106.68" x2="35.56" y2="106.68" width="0.1524" layer="91"/>
+<junction x="25.4" y="106.68"/>
+<pinref part="C80" gate="G$1" pin="1"/>
+<wire x1="35.56" y1="106.68" x2="45.72" y2="106.68" width="0.1524" layer="91"/>
+<junction x="35.56" y="106.68"/>
+<pinref part="C81" gate="G$1" pin="1"/>
+<wire x1="45.72" y1="106.68" x2="55.88" y2="106.68" width="0.1524" layer="91"/>
+<junction x="45.72" y="106.68"/>
+<pinref part="C82" gate="G$1" pin="1"/>
+<wire x1="55.88" y1="106.68" x2="66.04" y2="106.68" width="0.1524" layer="91"/>
+<junction x="55.88" y="106.68"/>
+<pinref part="C83" gate="G$1" pin="1"/>
+<wire x1="66.04" y1="106.68" x2="73.66" y2="106.68" width="0.1524" layer="91"/>
+<junction x="66.04" y="106.68"/>
+<pinref part="C56" gate="G$1" pin="1"/>
+<wire x1="73.66" y1="106.68" x2="81.28" y2="106.68" width="0.1524" layer="91"/>
+<junction x="73.66" y="106.68"/>
+<pinref part="SUPPLY37" gate="P" pin="+3.3V"/>
+<wire x1="81.28" y1="106.68" x2="81.28" y2="109.22" width="0.1524" layer="91"/>
+<junction x="81.28" y="106.68"/>
+</segment>
 </net>
 <net name="+1.8V" class="0">
@@
 </segment>
 </net>
-<net name="!CS!-RAD0" class="0">
+<net name="!CS!-RADIO" class="0">
 <segment>
 <pinref part="J2" gate="G$1" pin="5"/>
@@
 </segment>
 </net>
-<net name="INT-RAD0" class="0">
+<net name="INT-RADIO" class="0">
 <segment>
 <pinref part="J2" gate="G$1" pin="4"/>
@@
 </segment>
 </net>
-<net name="!CS!-IR" class="0">
+<net name="!CS!-WHISKERS" class="0">
 <segment>
 <pinref part="J1" gate="G$1" pin="4"/>
@@
 </segment>
 </net>
-<net name="!RST!-IR" class="0">
+<net name="!RST!-WHISKERS" class="0">
 <segment>
 <pinref part="J1" gate="G$1" pin="5"/>

Commit message: minor formatting changes
Other:
- note removed: "Pay attention to put the IMU board in the right pins while connecting"

Commit message: moved clock to sheet 3, removed busses in favor to individual signals
Parts:
- KIT2: value IMUIMU-KIT -> IMU; device RoboJackets-Boards:IMUIMU-KIT -> RoboJackets-Boards:IMU
Other:
- moved on the sheet: RN2, RN7, U8G$2
