File: boards/control-v3.5/control.sch (EAGLE design)
At the start: 150 parts, among them IC1 MCP23017-E/SS, J1 HFW8R-1ST, J2 HFW8R-1ST, J3 6-PIN_2MM-H, J4 HFW8R-1ST, J5 2-PIN-KICKERS, J6 DF22-2, Q1 BSS806NH6327XTSA1, Q2 BSS806NH6327XTSA1, U1 MCP1824T-1802E/OT, U2 SN74AHC1G125, U3 MPM3620GQV-P, U4 MPM3620GQV-P, U5 VND5E006ASPTR-E, U8 XC7A35T-1FTG256C, X1 ASV-50.000MHZ-E-T

Commit message: modifications after Arvind's review
Parts:
- added C9: 4.7uF, resistor:C-USC0603
- added D5: RED, RoboJackets-LEDs:LED-SMD-RED
- C24, C25: value GRM188R6YA106MA73D -> 10uF
- F1, F2: value 0805L200SLTHYR -> 2A
Connections:
- net !CS!-KICK renamed !CS!-KICKER
- net !CS!-WHISKERS renamed !CS!-SPI
- net !RST!-KICK renamed !RST!-KICKER
- net !RST!-WHISKERS renamed !RST!-SPI
- net SENSE-BATT renamed SENSE-BATTERY
- new net INT-SPI: J1G$1.6, KIT1.P12
- net +3.3V: now also D5.A, J1G$1.8
- net GND: now also C9.2
- net GVDD: now also C9.1
- net PWR-ERR: now also D5.K
- net VCCO_0: now also C9.1; no longer J1G$1.6
Other:
- note added: "SPI Connector"
- note removed: "IR Connector"
- moved on the sheet: D1

Commit message: don't remember which changes I did as they were forever ago but I did a thing last semester
Parts:
- renumbered U$17 to U6
Other:
- note added: "Add more I2C +SPI connections put some camera high speed connection from fpga bank"
- note added: "Change DC-DC converters to linear? needs more amp rating"
- note added: "INCREASE AMP RATING"
- note added: "RIGHT now VCC ADC enabled but connected to nothing, likely issues in how it is enabled, check datasheet"
Changed lines of the file:
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@@
 </instance>
 <instance part="C6" gate="G$1" x="104.14" y="137.16" smashed="yes" rot="R90">
-<attribute name="NAME" x="103.505" y="138.176" size="1.778" layer="95" rot="R90"/>
+<attribute name="NAME" x="103.505" y="140.716" size="1.778" layer="95" rot="R180"/>
 <attribute name="VALUE" x="107.696" y="138.049" size="1.778" layer="96"/>
 </instance>
 <instance part="C7" gate="G$1" x="104.14" y="121.92" smashed="yes" rot="R90">
-<attribute name="NAME" x="103.505" y="122.936" size="1.778" layer="95" rot="R90"/>
+<attribute name="NAME" x="103.505" y="125.476" size="1.778" layer="95" rot="R180"/>
 <attribute name="VALUE" x="107.696" y="122.809" size="1.778" layer="96"/>
 </instance>
 <instance part="C8" gate="G$1" x="104.14" y="106.68" smashed="yes" rot="R90">
-<attribute name="NAME" x="103.505" y="107.696" size="1.778" layer="95" rot="R90"/>
+<attribute name="NAME" x="103.505" y="110.236" size="1.778" layer="95" rot="R180"/>
 <attribute name="VALUE" x="107.696" y="107.569" size="1.778" layer="96"/>
 </instance>
@@
 <part name="U1" library="RoboJackets-PowerICs" deviceset="MCP1824T*?" device="OT" technology="-1802E/"/>
 <part name="SUPPLY6" library="RoboJackets-Supplies" deviceset="+1.8V" device=""/>
-<part name="U$17" library="RoboJackets-PowerICs" deviceset="MIC47100-1.0YML-TR" device=""/>
+<part name="U6" library="RoboJackets-PowerICs" deviceset="MIC47100-1.0YML-TR" device=""/>
 <part name="GND5" library="supply1" deviceset="GND" device=""/>
 <part name="C3" library="resistor" library_urn="urn:adsk.eagle:library:348" deviceset="C-US" device="C0603" package3d_urn="urn:adsk.eagle:package:23616/2" value="1uF"/>
@@
 <wire x1="266.7" y1="170.18" x2="165.1" y2="170.18" width="0.1524" layer="97" style="shortdash"/>
 <text x="167.64" y="165.1" size="1.778" layer="97">External Clock</text>
+<text x="-96.52" y="114.3" size="1.778" layer="97">RIGHT now VCC ADC enabled but
+connected to nothing, likely issues
+in how it is enabled, check datasheet</text>
 </plain>
 <instances>
@@
 |  HIGH  |     HIGH     ||  HIGH  |
 -------------------------------</text>
+<text x="172.72" y="111.76" size="1.778" layer="97">Add more I2C +SPI connections
+put some camera high speed connection from fpga bank</text>
 </plain>
 <instances>
@@
 <text x="38.1" y="55.88" size="1.778" layer="97">3.3V Regulator</text>
 <text x="208.28" y="109.22" size="1.778" layer="97">This part is fixed so pin 6 is FB</text>
+<text x="177.8" y="177.8" size="2.54" layer="97">Change DC-DC converters to linear? needs more amp rating </text>
+<text x="210.82" y="147.32" size="1.778" layer="97">INCREASE AMP RATING</text>
 </plain>
 <instances>
@@
 <attribute name="VALUE" x="231.775" y="81.915" size="1.778" layer="96"/>
 </instance>
-<instance part="U$17" gate="G$1" x="223.52" y="127" smashed="yes">
+<instance part="U6" gate="G$1" x="223.52" y="127" smashed="yes">
 <attribute name="NAME" x="210.82" y="140.716" size="1.778" layer="95"/>
 <attribute name="VALUE" x="210.82" y="116.84" size="1.778" layer="96"/>
@@
 <segment>
 <pinref part="GND9" gate="1" pin="GND"/>
-<pinref part="U$17" gate="G$1" pin="GND"/>
+<pinref part="U6" gate="G$1" pin="GND"/>
 <wire x1="203.2" y1="127" x2="205.74" y2="127" width="0.1524" layer="91"/>
 </segment>
@@
 <net name="+3.3V" class="0">
 <segment>
-<pinref part="U$17" gate="G$1" pin="BIAS"/>
+<pinref part="U6" gate="G$1" pin="BIAS"/>
 <pinref part="C3" gate="G$1" pin="1"/>
 <wire x1="205.74" y1="121.92" x2="200.66" y2="121.92" width="0.1524" layer="91"/>
@@
 </segment>
 <segment>
-<pinref part="U$17" gate="G$1" pin="EN"/>
+<pinref part="U6" gate="G$1" pin="EN"/>
 <pinref part="SUPPLY15" gate="P" pin="+3.3V"/>
 <wire x1="241.3" y1="121.92" x2="246.38" y2="121.92" width="0.1524" layer="91"/>
@@
 </segment>
 <segment>
-<pinref part="U$17" gate="G$1" pin="IN@0"/>
+<pinref part="U6" gate="G$1" pin="IN@0"/>
 <pinref part="C8" gate="G$1" pin="1"/>
 <wire x1="205.74" y1="137.16" x2="200.66" y2="137.16" width="0.1524" layer="91"/>
@@
 <net name="N$3" class="0">
 <segment>
-<pinref part="U$17" gate="G$1" pin="FB/ADJ"/>
+<pinref part="U6" gate="G$1" pin="FB/ADJ"/>
 <wire x1="241.3" y1="127" x2="246.38" y2="127" width="0.1524" layer="91"/>
-<pinref part="U$17" gate="G$1" pin="OUT@0"/>
+<pinref part="U6" gate="G$1" pin="OUT@0"/>
 <wire x1="241.3" y1="137.16" x2="246.38" y2="137.16" width="0.1524" layer="91"/>
 <wire x1="246.38" y1="137.16" x2="246.38" y2="132.08" width="0.1524" layer="91"/>
-<pinref part="U$17" gate="G$1" pin="OUT@1"/>
+<pinref part="U6" gate="G$1" pin="OUT@1"/>
 <wire x1="246.38" y1="132.08" x2="246.38" y2="127" width="0.1524" layer="91"/>
 <wire x1="241.3" y1="132.08" x2="246.38" y2="132.08" width="0.1524" layer="91"/>
