File: boards/control-v3.5/control.brd (EAGLE design)
At the start: 136.5 x 115.2 mm, 262 parts, among them IC1 MCP23017-E/SS, J1 HFW8R-1ST, J2 HFW8R-1ST, J3 6-PIN_2MM-H, J4 HFW8R-1ST, J5 2-PIN-KICKERS, J6 DF22-2, M1:C1 1uF, M1:C10 0.1uF 50V, M1:C12 ECA-1HHG221, M1:C13 ECA-1HHG221, M1:C2 1uF, M1:C3 0.022uF 50V, M1:C6 0.1uF 50V, M1:C7 0.1uF 50V, M1:C8 0.1uF 50V, M1:C9 2.2uF 50V, M1:J1 MKS-1658, M1:J2 4-PIN_2MM-H, M1:Q1 IRFH7545, M1:Q2 IRFH7545, M1:Q3 IRFH7545, M1:Q4 IRFH7545, M1:Q5 IRFH7545, M1:Q6 IRFH7545, M1:R1 10k, M1:U1 DRV8303DCA, M2:C1 1uF, M2:C10 0.1uF 50V, M2:C12 ECA-1HHG221, M2:C13 ECA-1HHG221, M2:C2 1uF, M2:C3 0.022uF 50V, M2:C6 0.1uF 50V, M2:C7 0.1uF 50V, M2:C8 0.1uF 50V, M2:C9 2.2uF 50V, M2:J1 MKS-1658, M2:J2 4-PIN_2MM-H, M2:Q1 IRFH7545, M2:Q2 IRFH7545, M2:Q3 IRFH7545, M2:Q4 IRFH7545, M2:Q5 IRFH7545, M2:Q6 IRFH7545, M2:R1 10k, M2:U1 DRV8303DCA, M3:C1 1uF, M3:C10 0.1uF 50V, M3:C12 ECA-1HHG221, M3:C13 ECA-1HHG221, M3:C2 1uF, M3:C3 0.022uF 50V, M3:C6 0.1uF 50V, M3:C7 0.1uF 50V, M3:C8 0.1uF 50V, M3:C9 2.2uF 50V, M3:J1 MKS-1658, M3:J2 4-PIN_2MM-H, M3:Q1 IRFH7545, M3:Q2 IRFH7545, M3:Q3 IRFH7545, M3:Q4 IRFH7545, M3:Q5 IRFH7545, M3:Q6 IRFH7545, M3:R1 10k, M3:U1 DRV8303DCA, M4:C1 1uF, M4:C10 0.1uF 50V, M4:C12 ECA-1HHG221, M4:C13 ECA-1HHG221, M4:C2 1uF, M4:C3 0.022uF 50V, M4:C6 0.1uF 50V, M4:C7 0.1uF 50V, M4:C8 0.1uF 50V, M4:C9 2.2uF 50V, M4:J1 MKS-1658, M4:J2 4-PIN_2MM-H, M4:Q1 IRFH7545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

Commit message: modifications after Arvind's review
Parts:
- added C9: 4.7uF, resistor:C0603
- added D5: RED, RoboJackets-LEDs:CHIP-LED0603
- C24, C25: value GRM188R6YA106MA73D -> 10uF
- F1, F2: value 0805L200SLTHYR -> 2A
Connections:
- net !CS!-KICK renamed !CS!-KICKER
- net !CS!-WHISKERS renamed !CS!-SPI
- net !RST!-KICK renamed !RST!-KICKER
- net !RST!-WHISKERS renamed !RST!-SPI
- net SENSE-BATT renamed SENSE-BATTERY
- new net INT-SPI: J1.6, KIT1.P$12
- net +3.3V: now also D5.A, J1.8
- net GND: now also C9.2
- net PWR-ERR: now also D5.C
- net VCCO_0: now also C9.1; no longer J1.6
Routing:
- net VCCO_0: track 60.6 -> 59.0 mm, vias 20 -> 19
- net GND: track 319.8 -> 318.9 mm

Commit message: don't remember which changes I did as they were forever ago but I did a thing last semester
Parts:
- renumbered U$17 to U6
Routing:
- net T25: track 0.00 -> 13.5 mm
- net T26: track 0.00 -> 12.2 mm
- net T27: track 0.00 -> 10.8 mm
- net T33: track 0.00 -> 9.82 mm
- net T29: track 0.00 -> 9.59 mm
- net T30: track 0.00 -> 9.50 mm
- net T28: track 0.00 -> 9.34 mm
- net T34: track 0.00 -> 8.59 mm
- net T38: track 0.00 -> 8.47 mm
- net T40: track 0.00 -> 8.45 mm
- net T32: track 0.00 -> 8.26 mm
- net T31: track 0.00 -> 8.01 mm
- net T35: track 0.00 -> 7.51 mm
- net T37: track 0.00 -> 7.30 mm
- net T39: track 0.00 -> 7.26 mm
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